Commit message: Make hardware async and update launch.py

File: example_17/description/ros2_control/mecanumwheelbot.ros2_control.xacro (robot description, xacro)
@@ -1,6 +1,6 @@
 <?xml version="1.0"?>
 <robot xmlns:xacro="http://www.ros.org/wiki/xacro">
-  <xacro:macro name="mecanumwheelbot_ros2_control" params="name prefix">
-    <ros2_control name="${name}" type="system">
+  <xacro:macro name="mecanumwheelbot_ros2_control" params="name prefix is_async:=false thread_priority:=1">
+    <ros2_control name="${name}" type="system" is_async="${is_async}" thread_priority="${thread_priority}">
       <hardware>
         <plugin>ros2_control_demo_example_17/MecanumWheelBotSystemHardware</plugin>

File: ros2_control_demo_description/mecanumwheelbot/urdf/mecanumwheelbot_description.urdf.xacro (robot description, xacro)
@@ -47,22 +47,4 @@
     </joint>
     <!-- rear wheels -->
-    <!-- virtual rear wheel -->
-    <!-- <link name="${prefix}virtual_rear_wheel">
-      <visual>
-        <origin xyz="0 0 0" rpy="${PI/2} 0 ${PI/2}"/>
-        <geometry>
-          <cylinder length="0.01" radius="${wheel_radius}"/>
-        </geometry>
-        <material name="invisible"/>
-      </visual>
-    </link> -->
-    <!-- <joint name="${prefix}virtual_rear_wheel_joint" type="continuous">
-      <parent link="${prefix}chassis_link"/>
-      <child link="${prefix}virtual_rear_wheel"/>
-      <origin xyz="-${wheelbase/2} 0 -${base_height/2}" rpy="0 0 ${PI/2}"/>
-      <axis xyz="1 0 0"/>
-      <limit effort="100.0" velocity="100.0"/>
-      <dynamics damping="0.2"/>
-    </joint> -->
     <!-- rear right wheel -->
     <link name="${prefix}rear_right_wheel">
@@ -93,8 +75,8 @@
       <child link="${prefix}rear_right_wheel"/>
       <origin xyz="-${wheelbase/2} ${base_width/2} -${base_height/2}" rpy="0 0 ${PI/2}"/>
-      <axis xyz="1 0 0"/>
+      <!-- Rollers angled +45° (forward and outward) -->
+      <axis xyz="1 1 0"/>
       <limit effort="100.0" velocity="100.0"/>
       <dynamics damping="0.2"/>
-      <!-- <mimic joint="${prefix}virtual_rear_wheel_joint" multiplier="1.0" offset="0.0"/> -->
     </joint>
     <!-- rear left wheel -->
@@ -126,28 +108,10 @@
       <child link="${prefix}rear_left_wheel" />
       <origin xyz="-${wheelbase/2} -${base_width/2} -${base_height/2}" rpy="0 0 ${PI/2}"/>
-      <axis xyz="1 0 0"/>
+      <!-- Rollers angled -45° (forward and inward) -->
+      <axis xyz="1 -1 0"/>
       <limit effort="100.0" velocity="100.0"/>
       <dynamics damping="0.2"/>
-      <!-- <mimic joint="${prefix}virtual_rear_wheel_joint" multiplier="1.0" offset="0.0"/> -->
     </joint>
     <!-- front wheels -->
-    <!-- virtual front wheel -->
-    <!-- <link name="${prefix}virtual_front_wheel">
-      <visual>
-        <origin xyz="0 0 0" rpy="${PI/2} 0 ${PI/2}"/>
-        <geometry>
-          <cylinder length="0.01" radius="${wheel_radius}"/>
-        </geometry>
-        <material name="invisible"/>
-      </visual>
-    </link> -->
-    <!-- <joint name="${prefix}virtual_front_wheel_joint" type="revolute">
-      <parent link="${prefix}chassis_link"/>
-      <child link="${prefix}virtual_front_wheel"/>
-      <origin xyz="${wheelbase/2} 0 -${base_height/2}" rpy="0 0 ${PI/2}"/>
-      <axis xyz="0 0 1"/>
-      <limit lower="-0.4" upper="0.4" effort="100.0" velocity="0.0"/>
-      <dynamics damping="0.2"/>
-    </joint> -->
     <!-- front right wheel -->
     <link name="${prefix}front_right_wheel">
@@ -178,8 +142,8 @@
       <child link="${prefix}front_right_wheel" />
       <origin xyz="${wheelbase/2} ${base_width/2} -${base_height/2}" rpy="0 0 ${PI/2}"/>
-      <axis xyz="0 0 1"/>
+      <!-- Rollers angled -45° (forward and inward) -->
+      <axis xyz="1 -1 0"/>
       <limit lower="-0.4" upper="0.4" effort="100.0" velocity="0.0"/>
       <dynamics damping="0.2"/>
-      <!-- <mimic joint="${prefix}virtual_front_wheel_joint" multiplier="1.0" offset="0.0"/> -->
     </joint>
     <!-- front left steering -->
@@ -211,8 +175,8 @@
       <child link="${prefix}front_left_wheel" />
       <origin xyz="${wheelbase/2} -${base_width/2} -${base_height/2}" rpy="0 0 ${PI/2}"/>
-      <axis xyz="0 0 1"/>
+      <!-- Rollers angled +45° (forward and outward) -->
+      <axis xyz="1 1 0"/>
       <limit lower="-0.4" upper="0.4" effort="100.0" velocity="0.0"/>
       <dynamics damping="0.2"/>
-      <!-- <mimic joint="${prefix}virtual_front_wheel_joint" multiplier="1.0" offset="0.0"/> -->
     </joint>
   </xacro:macro>

Commit message: Add rw_rate for async hardware

File: example_17/description/ros2_control/mecanumwheelbot.ros2_control.xacro (robot description, xacro)
@@ -1,6 +1,6 @@
 <?xml version="1.0"?>
 <robot xmlns:xacro="http://www.ros.org/wiki/xacro">
-  <xacro:macro name="mecanumwheelbot_ros2_control" params="name prefix is_async:=false thread_priority:=1">
-    <ros2_control name="${name}" type="system" is_async="${is_async}" thread_priority="${thread_priority}">
+  <xacro:macro name="mecanumwheelbot_ros2_control" params="name prefix is_async:=false thread_priority:=50 rw_rate:=0">
+    <ros2_control name="${name}" type="system" is_async="${is_async}" thread_priority="${thread_priority}" rw_rate="${rw_rate}">
       <hardware>
         <plugin>ros2_control_demo_example_17/MecanumWheelBotSystemHardware</plugin>
