Commit message: Initial check in for MecanumWheelBot

File: ros2_control_demo_description/mecanumwheelbot/urdf/mecanumwheelbot_description.urdf.xacro (robot description, xacro)
@@ -1,5 +1,5 @@
 <?xml version="1.0"?>
 <robot xmlns:xacro="http://www.ros.org/wiki/xacro">
-  <xacro:macro name="carlikebot" params="prefix">
+  <xacro:macro name="mecanumwheelbot" params="prefix">
   <!-- Constants for robot dimensions -->
   <xacro:property name="PI" value="3.1415926535897931"/>

Commit message: Update visual for mecanum wheels

File: ros2_control_demo_description/mecanumwheelbot/urdf/mecanumwheelbot_description.urdf.xacro (robot description, xacro)
@@ -56,7 +56,9 @@
       </collision>
       <visual>
-        <origin xyz="0 0 0" rpy="${PI/2} 0 ${PI/2}"/>
+        <!-- <origin xyz="0 0 0" rpy="${PI/2} 0 ${PI/2}"/> -->
+        <origin xyz="0 0 0" rpy="0 0 ${PI/2}"/>
         <geometry>
-          <cylinder length="${wheel_len}" radius="${wheel_radius}"/>
+          <!-- <cylinder length="${wheel_len}" radius="${wheel_radius}"/> -->
+          <mesh filename="package://ros2_control_demo_description/mecanumwheelbot/meshes/visual/rear_right.stl" scale="0.001 0.001 0.001"/>
         </geometry>
         <material name="black"/>
@@ -89,7 +91,9 @@
         </collision>
         <visual>
-          <origin xyz="0 0 0" rpy="${PI/2} 0 ${PI/2}"/>
+          <!-- <origin xyz="0 0 0" rpy="${PI/2} 0 ${PI/2}"/> -->
+          <origin xyz="0 0 0" rpy="0 0 ${PI/2}"/>
           <geometry>
-            <cylinder length="${wheel_len}" radius="${wheel_radius}"/>
+            <!-- <cylinder length="${wheel_len}" radius="${wheel_radius}"/> -->
+            <mesh filename="package://ros2_control_demo_description/mecanumwheelbot/meshes/visual/front_right.stl" scale="0.001 0.001 0.001"/>
           </geometry>
           <material name="black"/>
@@ -123,7 +127,9 @@
       </collision>
       <visual>
-        <origin xyz="0 0 0" rpy="${PI/2} 0 ${PI/2}"/>
+        <!-- <origin xyz="0 0 0" rpy="${PI/2} 0 ${PI/2}"/>   -->
+        <origin xyz="0 0 0" rpy="0 0 ${PI/2}"/>
         <geometry>
-          <cylinder length="${wheel_len}" radius="${wheel_radius}"/>
+          <!-- <cylinder length="${wheel_len}" radius="${wheel_radius}"/> -->
+          <mesh filename="package://ros2_control_demo_description/mecanumwheelbot/meshes/visual/front_right.stl" scale="0.001 0.001 0.001"/>
         </geometry>
         <material name="black"/>
@@ -156,7 +162,9 @@
       </collision>
       <visual>
-        <origin xyz="0 0 0" rpy="${PI/2} 0 ${PI/2}"/>
+        <!-- <origin xyz="0 0 0" rpy="${PI/2} 0 ${PI/2}"/> -->
+        <origin xyz="0 0 0" rpy="0 0 ${PI/2}"/>
         <geometry>
-          <cylinder length="${wheel_len}" radius="${wheel_radius}"/>
+          <!-- <cylinder length="${wheel_len}" radius="${wheel_radius}"/> -->
+          <mesh filename="package://ros2_control_demo_description/mecanumwheelbot/meshes/visual/rear_right.stl" scale="0.001 0.001 0.001"/>
         </geometry>
         <material name="black"/>

Commit message: Switch to use ros2_control_make

File: ros2_control_demo_description/mecanumwheelbot/urdf/mecanumwheelbot_description.urdf.xacro (robot description, xacro)
@@ -13,4 +13,7 @@
   <xacro:property name="wheel_radius" value="0.05" />
   <!-- <xacro:property name="wheeltrack" value="" -->
+  <!-- Define common wheel properties -->
+  <xacro:property name="wheel_effort_limit" value="10.0"/>
+  <xacro:property name="wheel_velocity_limit" value="5.0"/>
   <!-- Base Link -->
   <link name="${prefix}base_link" />
@@ -73,5 +76,5 @@
       </inertial>
     </link>
-    <joint name="${prefix}rear_right_wheel_joint" type="continuous">
+    <joint name="${prefix}rear_right_wheel_joint" type="revolute">
       <parent link="${prefix}chassis_link"/>
       <child link="${prefix}rear_right_wheel"/>
@@ -79,5 +82,5 @@
       <!-- Rollers angled +45° (forward and outward) -->
       <axis xyz="1 1 0"/>
-      <limit effort="100.0" velocity="100.0"/>
+      <limit effort="${wheel_effort_limit}" velocity="${wheel_velocity_limit}"/>
       <dynamics damping="0.2"/>
     </joint>
@@ -108,5 +111,5 @@
         </inertial>
     </link>
-    <joint name="${prefix}rear_left_wheel_joint" type="continuous">
+    <joint name="${prefix}rear_left_wheel_joint" type="revolute">
       <parent link="${prefix}chassis_link" />
       <child link="${prefix}rear_left_wheel" />
@@ -114,9 +117,9 @@
       <!-- Rollers angled -45° (forward and inward) -->
       <axis xyz="1 -1 0"/>
-      <limit effort="100.0" velocity="100.0"/>
+      <limit effort="${wheel_effort_limit}" velocity="${wheel_velocity_limit}"/>
       <dynamics damping="0.2"/>
     </joint>
     <!-- front wheels -->
-    <!-- front right wheel -->
+    <!-- front right wheel-->
     <link name="${prefix}front_right_wheel">
       <collision>
@@ -150,8 +153,8 @@
       <!-- Rollers angled -45° (forward and inward) -->
       <axis xyz="1 -1 0"/>
-      <limit lower="-0.4" upper="0.4" effort="100.0" velocity="0.0"/>
+      <limit lower="-0.4" upper="0.4" effort="${wheel_effort_limit}" velocity="${wheel_velocity_limit}"/>
       <dynamics damping="0.2"/>
     </joint>
-    <!-- front left steering -->
+    <!-- front left wheel -->
     <link name="${prefix}front_left_wheel">
       <collision>
@@ -185,5 +188,5 @@
       <!-- Rollers angled +45° (forward and outward) -->
       <axis xyz="1 1 0"/>
-      <limit lower="-0.4" upper="0.4" effort="100.0" velocity="0.0"/>
+      <limit lower="-0.4" upper="0.4" effort="${wheel_effort_limit}" velocity="${wheel_velocity_limit}"/>
       <dynamics damping="0.2"/>
     </joint>
