Commit message: Initial commit to support Gazebo sim

File: example_2/description/ros2_control/diffbot.ros2_control.xacro (robot description, xacro)
@@ -1,7 +1,7 @@
 <?xml version="1.0"?>
 <robot xmlns:xacro="http://www.ros.org/wiki/xacro">
-  <xacro:macro name="diffbot_ros2_control" params="name prefix use_mock_hardware">
+  <xacro:macro name="diffbot_ros2_control" params="name prefix  use_gazebo:=^|false">
     <ros2_control name="${name}" type="system">
-      <xacro:unless value="${use_mock_hardware}">
+      <xacro:unless value="${use_gazebo}">
         <hardware>
           <plugin>ros2_control_demo_example_2/DiffBotSystemHardware</plugin>
@@ -10,8 +10,7 @@
         </hardware>
       </xacro:unless>
-      <xacro:if value="${use_mock_hardware}">
+      <xacro:if value="${use_gazebo}">
         <hardware>
-          <plugin>mock_components/GenericSystem</plugin>
-          <param name="calculate_dynamics">true</param>
+          <plugin>gz_ros2_control/GazeboSimSystem</plugin>
         </hardware>
       </xacro:if>

File: example_2/description/urdf/diffbot.urdf.xacro (robot description, xacro)
@@ -3,5 +3,5 @@
 <robot xmlns:xacro="http://www.ros.org/wiki/xacro" name="diffdrive_robot">
   <xacro:arg name="prefix" default="" />
-  <xacro:arg name="use_mock_hardware" default="false" />
+  <xacro:arg name="use_gazebo" default="false" />
   <xacro:include filename="$(find ros2_control_demo_description)/diffbot/urdf/diffbot_description.urdf.xacro" />
   <!-- Import Rviz colors -->
@@ -11,4 +11,9 @@
   <xacro:diffbot prefix="$(arg prefix)" />
   <xacro:diffbot_ros2_control
-    name="DiffBot" prefix="$(arg prefix)" use_mock_hardware="$(arg use_mock_hardware)"/>
+    name="DiffBot" prefix="$(arg prefix)" use_gazebo="$(arg use_gazebo)"/>
+  <xacro:if value="$(arg use_gazebo)">
+    <!-- Import Gazebo definitions + plugin -->
+    <xacro:include filename="$(find ros2_control_demo_example_2)/gazebo/diffbot.gazebo.xacro" />
+    <xacro:diffbot_gazebo prefix="$(arg prefix)"/>
+  </xacro:if>
 </robot>
