Commit message: Updated with new control_msgs, still crashing

File: example_18/description/ros2_control/open_duck_mini.ros2_control.xacro (robot description, xacro)
@@ -2,5 +2,6 @@
 <robot xmlns:xacro="http://www.ros.org/wiki/xacro">
   <!--
-    Open Duck Mini ros2_control configuration for MuJoCo
+    Open Duck Mini ros2_control configuration
+    Supports both MuJoCo and mock hardware
     Total: 14 DoF (10 leg + 4 head)
     Joint order matches example_config.json joints_offsets (lines 13-28):
@@ -11,11 +12,22 @@
   -->
   <xacro:macro name="open_duck_mini_mujoco_ros2_control" params="name prefix">
+    <xacro:open_duck_mini_ros2_control name="${name}" prefix="${prefix}" use_mock_hardware="false"/>
+  </xacro:macro>
+  <xacro:macro name="open_duck_mini_ros2_control" params="name prefix use_mock_hardware:=^|false">
     <ros2_control name="${name}" type="system">
-      <hardware>
-        <plugin>mujoco_ros2_simulation/MujocoSystemInterface</plugin>
-        <param name="mujoco_model">$(find ros2_control_demo_example_18)/description/mujoco/scene.xml</param>
-        <param name="meshdir">$(find ros2_control_demo_example_18)/description/assets</param>
-        <param name="pids_config_file">$(find ros2_control_demo_example_18)/bringup/config/open_duck_mini_pids.yaml</param>
-      </hardware>
+      <xacro:unless value="${use_mock_hardware}">
+        <hardware>
+          <plugin>mujoco_ros2_simulation/MujocoSystemInterface</plugin>
+          <param name="mujoco_model">$(find ros2_control_demo_example_18)/description/mujoco/scene.xml</param>
+          <param name="meshdir">$(find ros2_control_demo_example_18)/description/assets</param>
+          <param name="pids_config_file">$(find ros2_control_demo_example_18)/bringup/config/open_duck_mini_pids.yaml</param>
+        </hardware>
+      </xacro:unless>
+      <xacro:if value="${use_mock_hardware}">
+        <hardware>
+          <plugin>mock_components/GenericSystem</plugin>
+          <param name="calculate_dynamics">true</param>
+        </hardware>
+      </xacro:if>
       <!-- Left leg joints -->
       <!-- Order matches example_config.json joints_offsets (lines 14-18) -->
@@ -153,6 +165,13 @@
       </joint>
       <!-- IMU sensor - matches Playground sensor names -->
-      <!-- MuJoCo sensors: gyro, accelerometer, velocimeter, framequat (orientation) -->
+      <!-- MuJoCo sensors: orientation (framequat), gyro, accelerometer -->
+      <!-- For mock hardware, sensor interfaces are still available but will return default values -->
       <sensor name="${prefix}imu">
+        <xacro:unless value="${use_mock_hardware}">
+          <param name="mujoco_type">imu</param>
+          <param name="mujoco_orientation_sensor">orientation</param>
+          <param name="mujoco_gyro_sensor">gyro</param>
+          <param name="mujoco_accel_sensor">accelerometer</param>
+        </xacro:unless>
         <state_interface name="orientation.w"/>
         <state_interface name="orientation.x"/>

File: example_18/description/urdf/open_duck_mini.urdf.xacro (robot description, xacro)
@@ -2,16 +2,17 @@
 <!-- Open Duck Mini Robot -->
 <!--
-This xacro file extends the base URDF with ros2_control configuration for MuJoCo.
+This xacro file extends the base URDF with ros2_control configuration.
 It includes the base robot description from robot.urdf
-and adds MuJoCo ros2_control plugin configuration.
+and adds ros2_control plugin configuration (supports both MuJoCo and mock hardware).
 -->
 <robot xmlns:xacro="http://www.ros.org/wiki/xacro" name="open-duck-mini">
   <xacro:arg name="prefix" default="" />
+  <xacro:arg name="use_mock_hardware" default="false" />
   <!-- Include the base URDF description -->
   <!-- Note: xacro will process the URDF file and merge its content -->
   <xacro:include filename="$(find ros2_control_demo_example_18)/description/mujoco/robot.urdf" />
-  <!-- Import Open Duck Mini MuJoCo ros2_control description -->
+  <!-- Import Open Duck Mini ros2_control description -->
   <xacro:include filename="$(find ros2_control_demo_example_18)/description/ros2_control/open_duck_mini.ros2_control.xacro" />
-  <xacro:open_duck_mini_mujoco_ros2_control
-    name="OpenDuckMini" prefix="$(arg prefix)"/>
+  <xacro:open_duck_mini_ros2_control
+    name="OpenDuckMini" prefix="$(arg prefix)" use_mock_hardware="$(arg use_mock_hardware)"/>
 </robot>
