Commit message: Add fune-tune support

File: example_18/description/mujoco/robot.urdf (robot description, URDF)
Before this commit: robot open-duck-mini, 16 links, 15 joints
Joints:
- joint head_pitch: limit lower=-0.78539816339744828 upper=0.78539816339744828 effort=3.23 velocity=10.0 -> lower=-10.0 upper=10.0 effort=3.23 velocity=10.0
- joint head_roll: limit lower=-0.52359877559821799 upper=0.52359877559837964 effort=3.23 velocity=10.0 -> lower=-10.0 upper=10.0 effort=3.23 velocity=10.0
- joint head_yaw: limit lower=-2.79252680319092716 upper=2.79252680319092716 effort=3.23 velocity=10.0 -> lower=-10.0 upper=10.0 effort=3.23 velocity=10.0
- joint left_ankle: limit lower=-1.57079632679489567 upper=1.57079632679489745 effort=3.23 velocity=10.0 -> lower=-10.0 upper=10.0 effort=3.23 velocity=10.0
- joint left_hip_pitch: limit lower=-1.22173047639603061 upper=0.52359877559829882 effort=3.23 velocity=10.0 -> lower=-10.0 upper=10.0 effort=3.23 velocity=10.0
- joint left_hip_roll: limit lower=-0.43633231299858150 upper=0.43633231299858327 effort=3.23 velocity=10.0 -> lower=-10.0 upper=10.0 effort=3.23 velocity=10.0
- joint left_hip_yaw: limit lower=-0.52359877559829793 upper=0.52359877559829970 effort=3.23 velocity=10.0 -> lower=-10.0 upper=10.0 effort=3.23 velocity=10.0
- joint left_knee: limit lower=-1.57079632679489656 upper=1.57079632679489656 effort=3.23 velocity=10.0 -> lower=-10.0 upper=10.0 effort=3.23 velocity=10.0
- joint neck_pitch: limit lower=-0.34906585039884369 upper=1.13446401379633643 effort=3.23 velocity=10.0 -> lower=-10.0 upper=10.0 effort=3.23 velocity=10.0
- joint right_ankle: limit lower=-1.57079632679489567 upper=1.57079632679489745 effort=3.23 velocity=10.0 -> lower=-10.0 upper=10.0 effort=3.23 velocity=10.0
- joint right_hip_pitch: limit lower=-0.52359877559829882 upper=1.22173047639603061 effort=3.23 velocity=10.0 -> lower=-10.0 upper=10.0 effort=3.23 velocity=10.0
- joint right_knee: limit lower=-1.57079632679489656 upper=1.57079632679489656 effort=3.23 velocity=10.0 -> lower=-10.0 upper=10.0 effort=3.23 velocity=10.0

File: example_18/description/ros2_control/open_duck_mini.ros2_control.xacro (robot description, xacro)
@@ -21,5 +21,7 @@
           <param name="mujoco_model">$(find ros2_control_demo_example_18)/description/mujoco/scene.xml</param>
           <param name="meshdir">$(find ros2_control_demo_example_18)/description/assets</param>
-          <param name="pids_config_file">$(find ros2_control_demo_example_18)/config/open_duck_mini_pids.yaml</param>
+          <!-- DISABLED: Using MuJoCo's built-in position actuators (kp=13.37) instead of external PID -->
+          <!-- External PID adds loop delay and numerical differences compared to Python reference -->
+          <!-- <param name="pids_config_file">$(find ros2_control_demo_example_18)/config/open_duck_mini_pids.yaml</param> -->
           <!-- Initialize robot from "home" keyframe to match reference implementation -->
           <!-- Source: scene_flat_terrain.xml keyframe "home" -->
@@ -37,6 +39,7 @@
       <joint name="${prefix}left_hip_yaw">
         <command_interface name="position">
-          <param name="min">-0.52359877559829881566</param>
-          <param name="max">0.52359877559829881566</param>
+          <!-- Joint limits set to very large values for data collection - reference motion may exceed URDF limits -->
+          <param name="min">-10.0</param>
+          <param name="max">10.0</param>
         </command_interface>
         <state_interface name="position"/>
@@ -46,6 +49,7 @@
       <joint name="${prefix}left_hip_roll">
         <command_interface name="position">
-          <param name="min">-0.43633231299858238339</param>
-          <param name="max">0.43633231299858238339</param>
+          <!-- Joint limits set to very large values for data collection -->
+          <param name="min">-10.0</param>
+          <param name="max">10.0</param>
         </command_interface>
         <state_interface name="position"/>
@@ -55,6 +59,6 @@
       <joint name="${prefix}left_hip_pitch">
         <command_interface name="position">
-          <param name="min">-1.2217304763960306069</param>
-          <param name="max">0.52359877559829881566</param>
+          <param name="min">-10.0</param>
+          <param name="max">10.0</param>
         </command_interface>
         <state_interface name="position"/>
@@ -64,6 +68,6 @@
       <joint name="${prefix}left_knee">
         <command_interface name="position">
-          <param name="min">-1.570796326794896558</param>
-          <param name="max">1.570796326794896558</param>
+          <param name="min">-10.0</param>
+          <param name="max">10.0</param>
         </command_interface>
         <state_interface name="position"/>
@@ -73,6 +77,6 @@
       <joint name="${prefix}left_ankle">
         <command_interface name="position">
-          <param name="min">-1.570796326794896558</param>
-          <param name="max">1.570796326794896558</param>
+          <param name="min">-10.0</param>
+          <param name="max">10.0</param>
         </command_interface>
         <state_interface name="position"/>
@@ -86,6 +90,6 @@
       <joint name="${prefix}neck_pitch">
         <command_interface name="position">
-          <param name="min">-0.3490658503988437</param>  <!-- ~-20 degrees -->
-          <param name="max">1.1344640137963364</param>   <!-- ~65 degrees -->
+          <param name="min">-10.0</param>
+          <param name="max">10.0</param>
         </command_interface>
         <state_interface name="position"/>
@@ -95,6 +99,6 @@
       <joint name="${prefix}head_pitch">
         <command_interface name="position">
-          <param name="min">-0.785398163397448279</param>  <!-- -45 degrees -->
-          <param name="max">0.785398163397448279</param>   <!-- +45 degrees -->
+          <param name="min">-10.0</param>
+          <param name="max">10.0</param>
         </command_interface>
         <state_interface name="position"/>
@@ -104,6 +108,6 @@
       <joint name="${prefix}head_yaw">
         <command_interface name="position">
-          <param name="min">-2.792526803190927</param>  <!-- ~-160 degrees -->
-          <param name="max">2.792526803190927</param>   <!-- ~+160 degrees -->
+          <param name="min">-10.0</param>
+          <param name="max">10.0</param>
         </command_interface>
         <state_interface name="position"/>
@@ -113,6 +117,6 @@
       <joint name="${prefix}head_roll">
         <command_interface name="position">
-          <param name="min">-0.523598775598218</param>  <!-- ~-30 degrees -->
-          <param name="max">0.5235987755983796</param>   <!-- ~+30 degrees -->
+          <param name="min">-10.0</param>
+          <param name="max">10.0</param>
         </command_interface>
         <state_interface name="position"/>
@@ -124,6 +128,6 @@
       <joint name="${prefix}right_hip_yaw">
         <command_interface name="position">
-          <param name="min">-0.52359877559829881566</param>
-          <param name="max">0.52359877559829881566</param>
+          <param name="min">-10.0</param>
+          <param name="max">10.0</param>
         </command_interface>
         <state_interface name="position"/>
@@ -133,6 +137,6 @@
       <joint name="${prefix}right_hip_roll">
         <command_interface name="position">
-          <param name="min">-0.43633231299858238339</param>
-          <param name="max">0.43633231299858238339</param>
+          <param name="min">-10.0</param>
+          <param name="max">10.0</param>
         </command_interface>
         <state_interface name="position"/>
@@ -142,6 +146,6 @@
       <joint name="${prefix}right_hip_pitch">
         <command_interface name="position">
-          <param name="min">-0.52359877559829881566</param>
-          <param name="max">1.2217304763960306069</param>
+          <param name="min">-10.0</param>
+          <param name="max">10.0</param>
         </command_interface>
         <state_interface name="position"/>
@@ -151,6 +155,6 @@
       <joint name="${prefix}right_knee">
         <command_interface name="position">
-          <param name="min">-1.570796326794896558</param>
-          <param name="max">1.570796326794896558</param>
+          <param name="min">-10.0</param>
+          <param name="max">10.0</param>
         </command_interface>
         <state_interface name="position"/>
@@ -160,6 +164,6 @@
       <joint name="${prefix}right_ankle">
         <command_interface name="position">
-          <param name="min">-1.570796326794896558</param>
-          <param name="max">1.570796326794896558</param>
+          <param name="min">-10.0</param>
+          <param name="max">10.0</param>
         </command_interface>
         <state_interface name="position"/>
@@ -188,4 +192,36 @@
         <state_interface name="linear_acceleration.z"/>
       </sensor>
+      <!-- Velocimeter sensor - base linear velocity in local frame -->
+      <!-- MuJoCo sensor: velocimeter (local_linvel) -->
+      <!-- Provides 3D linear velocity of the base in the local frame -->
+      <sensor name="${prefix}velocimeter">
+        <xacro:unless value="${use_mock_hardware}">
+          <param name="mujoco_type">velocimeter</param>
+          <param name="mujoco_sensor_name">local_linvel</param>
+        </xacro:unless>
+        <state_interface name="linear_velocity.x"/>
+        <state_interface name="linear_velocity.y"/>
+        <state_interface name="linear_velocity.z"/>
+      </sensor>
+      <!-- Contact sensors - MuJoCo collision detection -->
+      <!-- Reference: Python mujoco_infer_base.py get_feet_contacts() (lines 280-283) -->
+      <!-- Checks collisions between foot bodies and floor using mj_data_->contact[] array -->
+      <!-- Matches Python reference: check_contact(data, "foot_assembly", "floor") -->
+      <sensor name="${prefix}left_foot_contact">
+        <xacro:unless value="${use_mock_hardware}">
+          <param name="mujoco_type">contact</param>
+          <param name="body1_name">foot_assembly</param>
+          <param name="body2_name">floor</param>
+        </xacro:unless>
+        <state_interface name="contact"/>
+      </sensor>
+      <sensor name="${prefix}right_foot_contact">
+        <xacro:unless value="${use_mock_hardware}">
+          <param name="mujoco_type">contact</param>
+          <param name="body1_name">foot_assembly_2</param>
+          <param name="body2_name">floor</param>
+        </xacro:unless>
+        <state_interface name="contact"/>
+      </sensor>
     </ros2_control>
   </xacro:macro>
